File: PicoShield_B8/PicoShield.kicad_pcb (KiCad board)
At the start: 2 copper layers, 55.8 x 53.8 mm, 25 parts, among them J1 Conn_02x04_Counter_Clockwise, J2 Conn_02x04_Counter_Clockwise, J4 Conn_02x04_Counter_Clockwise, J5 Conn_02x04_Counter_Clockwise, J6 Conn_02x04_Counter_Clockwise, J8 Micro_SD_Card_Det2, U1 74LVC125, U2 AT45DB641E

Commit message: Correction DLC
Other:
- board text added: "B8"
Changed lines of the file:
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@@
 			(plot_on_all_layers_selection 0x0000000_00000000)
 			(disableapertmacros no)
-			(usegerberextensions no)
+			(usegerberextensions yes)
 			(usegerberattributes yes)
 			(usegerberadvancedattributes yes)
@@
 			(drillshape 0)
 			(scaleselection 1)
-			(outputdirectory "GerberPicoShield")
+			(outputdirectory "PICOB8/")
 		)
 	)
@@
 		(tags "SOIC SO")
 		(property "Reference" "U2"
-			(at 0 3.59 360)
+			(at 0 3.59 0)
 			(layer "B.SilkS")
 			(effects
@@
 		)
 		(property "Value" "AT45DB641E"
-			(at 0 -3.59 360)
+			(at 0 -3.59 0)
 			(layer "B.Fab")
 			(effects
@@
 		)
 		(fp_text user "${REFERENCE}"
-			(at 0 0 360)
+			(at 0 0 0)
 			(layer "B.Fab")
 			(effects
@@
 		(layer "Edge.Cuts")
 	)
+	(gr_text "B8"
+		(at 131.6736 75.1332 0)
+		(layer "F.SilkS")
+		(effects
+			(font
+				(size 1 1)
+				(thickness 0.15)
+			)
+			(justify left bottom)
+		)
+	)
 	(segment
 		(start 133.731 51.16)
@@
 		(layer "B.Cu")
 		(net 4)
-	)
-	(segment
-		(start 144.9125 56.4125)
-		(end 145 56.5)
-		(width 0.25)
-		(layer "B.Cu")
-		(net 4)
