File: PicoMother/PicoMother.kicad_pcb (KiCad board)
At the start: 2 copper layers, 66 x 53.3 mm, 61 parts, among them J1 M20-9980345, J2 Micro_SD_Card_Det2, J3 M20-9980345, J4 Conn_02x04_Counter_Clockwise, J5 Conn_02x04_Counter_Clockwise, J6 Conn_02x04_Counter_Clockwise, J7 Conn_02x04_Counter_Clockwise, J8 USB_C_Receptacle_USB2.0_16P, J9 Conn_02x04_Counter_Clockwise, SW1 SW_Push, U1 74LVC125, U3 ATMEGA16U2-MU, U4 ATMEGA328P-MU, Y1 CSTNE16M0V530000R0, Y2 LFXTAL003240BULK

Commit message: avancement schema
Parts:
- removed C6: 100n, Capacitor_SMD:C_0603_1608Metric
- moved U4 28.1 mm to (150.8, 113.2)
- moved J2 17.1 mm to (104.5, 119.2)
Connections:
- net IO0 renamed Net-(U4-PD0)
- R7 pad 2: IO1 -> CS4
- U4 pad 1: IO3 -> INT3
- U4 pad 10: IO6 -> INT4
- U4 pad 11: IO7 -> CS6
- U4 pad 12: IO8 -> RST5
- U4 pad 13: IO9 -> INT5
- U4 pad 14: SS -> CS1
- U4 pad 2: IO4 -> CS5
- U4 pad 23: A0 -> CS2
- U4 pad 24: A1 -> RST1
- U4 pad 25: A2 -> INT1
- U4 pad 26: A3 -> CS3
- U4 pad 27: A4/SDA -> RST2
- U4 pad 28: A5/SCL -> INT2
- U4 pad 31: IO1 -> CS4
- U4 pad 32: IO2 -> RST3
- U4 pad 9: IO5 -> RST4
Other:
- board outline removed

Commit message: Schema PicoMother
Parts:
- removed D2, D3: CD1206-S01575, Diode_SMD:D_1206_3216Metric
- removed FB1: 1kΩ@100MHz, Inductor_SMD:L_0805_2012Metric
- removed FB2: 10uH, Inductor_SMD:L_0805_2012Metric
- removed Z1, Z2: 5pF@1MHz, Resistor_SMD:R_0603_1608Metric
- added C2: 100nF, Capacitor_SMD:C_0603_1608Metric_Pad1.08x0.95mm_HandSolder, F.Cu at (142.9, 53.9)
- added C3: 100nF, Capacitor_SMD:C_0603_1608Metric_Pad1.08x0.95mm_HandSolder, F.Cu at (142.9, 56.4)
- added U2: LM1117-3.3, Package_TO_SOT_SMD:SOT-23, F.Cu at (147.6, 55.0)
- C1, C10, C11, C12, C13, C7, C8, C9: footprint Capacitor_SMD:C_0603_1608Metric -> Capacitor_SMD:C_0603_1608Metric_Pad1.08x0.95mm_HandSolder
- D1, D5, D6: footprint LED_SMD:LED_0805_2012Metric -> LED_SMD:LED_0603_1608Metric_Pad1.05x0.95mm_HandSolder
- R1, R2, R3, R4: footprint Resistor_SMD:R_0603_1608Metric -> Resistor_SMD:R_0603_1608Metric_Pad0.98x0.95mm_HandSolder
- U3: value ATMEGA16U2-MU -> ATMEGA8U2-MU
- Y1: value CSTNE16M0V530000R0 -> 16Mhz; footprint Crystal:Resonator_SMD_Murata_CSTxExxV-3Pin_3.0x1.1mm -> Crystal:Crystal_SMD_SeikoEpson_FA238-4Pin_3.2x2.5mm_HandSoldering
- Y2: value LFXTAL003240BULK -> 16Mhz; footprint Crystal:Crystal_HC49-4H_Vertical -> Crystal:Crystal_SMD_SeikoEpson_FA238-4Pin_3.2x2.5mm_HandSoldering
- moved C13 71.4 mm to (65.0, 102.5)
- moved C7 70.8 mm to (71.4, 100.0)
- moved R1 68.3 mm to (65.0, 105.0), turned to 0 degrees
- moved C11 65.2 mm to (65.0, 100.0), turned to 0 degrees
Connections:
- J8 pad S1: USHIELD -> GND
Routing:
- net Net-(U3-PC0): track 8.18 -> 0.00 mm
- net Net-(U3-XTAL1): track 7.84 -> 0.00 mm

Commit message: Premier Schema
Parts:
- D1: value GREEN -> LED
- D5, D6: value YELLOW -> LED
- J2: value Micro_SD_Card_Det2 -> Micro_SD
- J8: value USB_C_Receptacle_USB2.0_16P -> USB_C
- moved D1 74.1 mm to (132.4, 107.0)
- moved C1 74.1 mm to (132.1, 111.8)
- moved C2 73.4 mm to (127.6, 125.7)
- moved U2 73.4 mm to (132.2, 126.8)
- moved C3 73.4 mm to (127.6, 128.2)
- moved SW1 67.1 mm to (164.5, 87.1), turned to -90 degrees
- moved C11 56.1 mm to (119.6, 113.2)
- moved C13 56.1 mm to (119.6, 115.7)
- moved R1 56.1 mm to (119.6, 118.2)
- moved C7 56.1 mm to (125.9, 113.2)
- moved J2 53.4 mm to (157.5, 125.5), turned to 180 degrees
- moved Y1 44.4 mm to (148.2, 100.5)
- moved J3 39.6 mm to (161.7, 105.5)
- moved U1 34.6 mm to (145.5, 124.8)
- moved D4 34.6 mm to (139.1, 120.8)
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Connections:
- net AREF renamed Net-(U4-AREF)
- net AVCC renamed Net-(U4-AVCC)
- D1 pad 1: GND -> Net-(D1-K)
- D1 pad 2: Net-(D1-A) -> GND
- J1 pad 2: +5V -> RESET2
- J8 pad A4: USBVCC -> +5V
- J8 pad A6: D+ -> Net-(J8-D+-PadA6)
- J8 pad A7: D- -> Net-(J8-D--PadA7)
- J8 pad A9: USBVCC -> +5V
- J8 pad B4: USBVCC -> +5V
- J8 pad B6: D+ -> Net-(J8-D+-PadA6)
- J8 pad B7: D- -> Net-(J8-D--PadA7)
- J8 pad B9: USBVCC -> +5V
- R11 pad 1: D- -> Net-(J8-D--PadA7)
- R11 pad 2: RD- -> D-
- R12 pad 1: D+ -> Net-(J8-D+-PadA6)
- R12 pad 2: RD+ -> D+
- R6 pad 2: Net-(D1-A) -> Net-(D1-K)
- U3 pad 29: RD+ -> D+
- U3 pad 30: RD- -> D-
Other:
- board text removed: "ICSP"

Commit message: correction schematique quartz
Parts:
- removed Y1, Y2: 16Mhz, Crystal:Crystal_SMD_SeikoEpson_FA238-4Pin_3.2x2.5mm_HandSoldering
- added C4: 22p, Capacitor_SMD:C_0603_1608Metric_Pad1.08x0.95mm_HandSolder, F.Cu at (103.5, 118.2)
- added C5: 22p, Capacitor_SMD:C_0603_1608Metric_Pad1.08x0.95mm_HandSolder, F.Cu at (103.5, 120.7)
- added Y3: Crystal_GND24, Crystal:Crystal_SMD_SeikoEpson_FA238-4Pin_3.2x2.5mm_HandSoldering, F.Cu at (139.1, 106.7)
- added Y4: Crystal_GND24, Crystal:Crystal_SMD_SeikoEpson_FA238-4Pin_3.2x2.5mm_HandSoldering, F.Cu at (132.1, 95.1)
- moved J1 2.10 mm to (124.6, 79.0)

Commit message: correction schematique reset
Parts:
- moved R8 9.06 mm to (158.5, 93.0)
- moved J1 7.72 mm to (117.2, 81.5), turned to 90 degrees
Connections:
- J1 pad 2: RESET2 -> +5V
Routing:
- net RESET2: track 0.00 -> 16.8 mm, vias 0 -> 1
- net MOSI2: track 0.00 -> 9.96 mm
- net MISO2: track 0.00 -> 8.24 mm
- net SCK2: track 0.00 -> 6.91 mm

Commit message: correction schematique empreintes MCU
Parts:
- removed C10: 1u, Capacitor_SMD:C_0603_1608Metric_Pad1.08x0.95mm_HandSolder
- removed C12, C8: 100n, Capacitor_SMD:C_0603_1608Metric_Pad1.08x0.95mm_HandSolder
- removed U3: ATMEGA8U2-MU, Package_QFP:TQFP-32_7x7mm_P0.8mm
- removed Y3: Crystal_GND24, Crystal:Crystal_SMD_SeikoEpson_FA238-4Pin_3.2x2.5mm_HandSoldering
- added C6: 100n, Capacitor_SMD:C_0603_1608Metric_Pad1.08x0.95mm_HandSolder, F.Cu at (101.6, 132.6)
- added U5: ATmega8U2-A, Package_QFP:TQFP-32_7x7mm_P0.8mm, F.Cu at (121.5, 92.6)
- added Y1: Crystal_GND24, Crystal:Crystal_SMD_SeikoEpson_FA238-4Pin_3.2x2.5mm_HandSoldering, F.Cu at (117.3, 138.2)
- C7: value 100n -> 1u
- R2: value 1M -> 1k
- R7: value 1k -> 1M
- SW1: footprint Button_Switch_THT:SW_DIP_SPSTx01_Piano_10.8x4.1mm_W7.62mm_P2.54mm -> Button_Switch_SMD:SW_Push_1P1T_NO_CK_KSC7xxJ
- U4: value ATMEGA328P-MU -> ATmega328P-A
- moved R7 118.9 mm to (101.6, 140.1)
- moved R5 118.9 mm to (101.6, 137.6)
- moved R6 110.9 mm to (110.8, 144.6)
- moved R13 79.6 mm to (101.6, 142.6)
- moved R14 79.6 mm to (101.6, 145.1)
- moved SW1 76.3 mm to (108.9, 139.3), turned to 0 degrees
- moved R2 45.8 mm to (101.6, 135.1)
- moved R8 45.0 mm to (113.5, 94.6), turned to 180 degrees
- moved U4 44.8 mm to (109.6, 129.6), turned to 0 degrees
- moved D1 40.7 mm to (91.6, 106.1)
- moved C1 33.3 mm to (101.6, 125.0)
- moved C13 27.7 mm to (132.2, 91.1)
- moved R1 24.9 mm to (128.3, 94.9), turned to -90 degrees
- moved C7 20.3 mm to (113.5, 97.1), turned to 180 degrees
- moved C11 18.9 mm to (132.2, 99.2), turned to 180 degrees
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Connections:
- C1 pad 1: Net-(U4-AREF) -> DTR
- C1 pad 2: GND -> RESET
- C2 pad 1: +5V -> USBVCC
- C4 pad 1: Net-(U4-PB7) -> Net-(U4-XTAL1/PB6)
- C5 pad 1: Net-(U4-PB6) -> Net-(U4-XTAL2/PB7)
- C7 pad 1: DTR -> GND
- C7 pad 2: RESET -> Net-(U5-UCAP)
- C9 pad 1: +5V -> USBVCC
- J1 pad 2: +5V -> USBVCC
- J3 pad 2: +5V -> USBVCC
- J4 pad 2: +5V -> USBVCC
- J5 pad 2: +5V -> USBVCC
- J6 pad 2: +5V -> USBVCC
- J7 pad 2: +5V -> USBVCC
- J8 pad A4: +5V -> USBVCC
- J8 pad A9: +5V -> USBVCC
- J8 pad B4: +5V -> USBVCC
- J8 pad B9: +5V -> USBVCC
- J9 pad 2: +5V -> USBVCC
- R10 pad 2: +5V -> USBVCC
- R14 pad 1: +5V -> USBVCC
- R2 pad 1: Net-(U4-PB7) -> CS4
- R2 pad 2: Net-(U4-PB6) -> M8RXD
- R5 pad 1: Net-(U4-PD0) -> M8TXD
- R5 pad 2: M8RXD -> Net-(U4-PD1)
- R6 pad 1: +5V -> USBVCC
- R7 pad 1: M8TXD -> Net-(U4-XTAL1/PB6)
- R7 pad 2: CS4 -> Net-(U4-XTAL2/PB7)
- R8 pad 1: +5V -> USBVCC
- R9 pad 2: +5V -> USBVCC
- U2 pad 3: +5V -> USBVCC
- U4 pad 18: Net-(U4-AVCC) -> USBVCC
- U4 pad 20: Net-(U4-AREF) -> unconnected-(U4-AREF-Pad20)
- U4 pad 21: GND -> Net-(U4-GND-Pad21)
- U4 pad 3: GND -> Net-(U4-GND-Pad21)
- U4 pad 30: Net-(U4-PD0) -> CS4
- U4 pad 31: CS4 -> Net-(U4-PD1)
- U4 pad 4: +5V -> USBVCC
- U4 pad 5: GND -> Net-(U4-GND-Pad21)
- U4 pad 6: +5V -> USBVCC
- U4 pad 7: Net-(U4-PB6) -> Net-(U4-XTAL1/PB6)
- U4 pad 8: Net-(U4-PB7) -> Net-(U4-XTAL2/PB7)
Routing:
- net Net-(U5-PC0/XTAL2): track 0.00 -> 12.3 mm
- net Net-(U5-XTAL1): track 0.00 -> 10.6 mm
Other:
- board text removed: "RESET"

Commit message: début de routage, placement encore perfectible
Parts:
- moved SW1 65.4 mm to (141.3, 82.5), turned to 90 degrees
- moved R15 64.5 mm to (155.2, 78.0)
- moved R16 64.5 mm to (155.2, 80.6)
- moved R17 64.5 mm to (155.2, 83.1)
- moved R18 64.5 mm to (155.2, 85.6)
- moved R19 64.5 mm to (155.2, 88.1)
- moved R20 64.5 mm to (155.2, 90.6)
- moved R22 64.5 mm to (155.2, 95.6)
- moved R23 64.5 mm to (155.2, 98.1)
- moved R21 64.5 mm to (155.2, 93.1)
- moved R10 42.2 mm to (111.4, 80.2)
- moved R9 42.2 mm to (111.4, 77.7)
- moved R5 40.6 mm to (117.9, 100.4), turned to -90 degrees
- moved J3 39.5 mm to (124.7, 119.1), turned to -90 degrees
- moved R2 39.4 mm to (120.2, 100.4), turned to 90 degrees
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Routing:
- net DTR: track 0.00 -> 18.4 mm, vias 0 -> 2
- net M8TXD: track 0.00 -> 16.7 mm, vias 0 -> 2
- net M8RXD: track 0.00 -> 12.8 mm, vias 0 -> 2
- net RESET: track 0.00 -> 4.33 mm
- net Net-(U4-PD1): track 0.00 -> 4.26 mm
- net CS4: track 0.00 -> 3.22 mm
Other:
- board text removed: "ON"

Commit message: début de routage, meilleur placement, encore perfectible
Parts:
- moved R13 49.4 mm to (134.7, 86.6)
- moved J3 40.6 mm to (143.0, 82.9), turned to 90 degrees
- moved C5 39.7 mm to (147.8, 102.1), turned to -90 degrees
- moved Y1 35.4 mm to (143.6, 102.5), turned to 180 degrees
- moved R7 32.2 mm to (143.5, 98.7), turned to 0 degrees
- moved SW1 30.3 mm to (138.3, 112.7)
- moved C4 28.1 mm to (139.4, 102.2)
- moved U4 25.6 mm to (141.1, 92.1), turned to 90 degrees
- moved R10 22.8 mm to (132.6, 88.4), turned to 90 degrees
- moved R9 21.6 mm to (130.5, 87.7), turned to 90 degrees
- moved D1 21.5 mm to (109.4, 118.2)
- moved R4 18.0 mm to (112.1, 99.1), turned to -90 degrees
- moved C9 17.7 mm to (113.0, 89.7), turned to 180 degrees
- moved R8 16.8 mm to (120.4, 81.2), turned to -90 degrees
- moved C11 16.0 mm to (116.6, 102.8), turned to 90 degrees
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Routing:
- net DTR: track 18.4 -> 0.00 mm, vias 2 -> 0
- net RESET2: track 16.8 -> 0.00 mm, vias 1 -> 0
- net M8TXD: track 16.7 -> 0.00 mm, vias 2 -> 0
- net M8RXD: track 12.8 -> 0.00 mm, vias 2 -> 0
- net MOSI2: track 9.96 -> 0.00 mm
- net MISO2: track 8.24 -> 0.00 mm
- net SCK2: track 6.91 -> 0.00 mm
- net RESET: track 4.33 -> 0.00 mm
- net Net-(U4-PD1): track 4.26 -> 0.00 mm
- net CS4: track 3.22 -> 0.00 mm
Other:
- board text removed: "RX"
- board text removed: "TX"
