File: PicoMother/PicoMother.kicad_pcb (KiCad board)
At the start: 2 copper layers, 57 parts, among them J1 M20-9980345, J2 Micro_SD, J3 M20-9980345, J4 Conn_02x04_Counter_Clockwise, J5 Conn_02x04_Counter_Clockwise, J6 Conn_02x04_Counter_Clockwise, J7 Conn_02x04_Counter_Clockwise, J8 USB_C, J9 Conn_02x04_Counter_Clockwise, SW1 SW_Push, U1 74LVC125, U2 LM1117-3.3, U4 ATmega328P-A, U5 ATmega8U2-A, Y1 Crystal_GND24, Y4 Crystal_GND24

Commit message: placement des composants pratiquement stable
Parts:
- moved R17 49.3 mm to (116.8, 113.9), turned to 90 degrees
- moved R23 48.9 mm to (112.1, 121.3), turned to -90 degrees
- moved J9 48.5 mm to (120.0, 123.2)
- moved R16 47.3 mm to (116.9, 108.3), turned to -90 degrees
- moved R15 46.4 mm to (127.2, 115.1), turned to 90 degrees
- moved J2 42.0 mm to (107.7, 110.8), turned to 90 degrees
- moved D10 40.6 mm to (112.1, 125.2), turned to 90 degrees
- moved R18 38.0 mm to (127.2, 111.3), turned to 90 degrees
- moved C6 38.0 mm to (136.1, 101.3)
- moved U1 35.8 mm to (121.9, 111.7)
- moved J7 28.6 mm to (140.4, 123.3)
- moved R22 25.9 mm to (155.1, 121.5), turned to -90 degrees
- moved R6 25.5 mm to (108.8, 100.6), turned to 180 degrees
- moved C2 24.5 mm to (131.0, 101.4), turned to 180 degrees
- moved U2 21.2 mm to (131.1, 105.6), turned to 90 degrees
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
Commit message: début de routage, premiers changement d'E/S sur le 328 pour faciliter le routage
Parts:
- moved C9 13.5 mm to (108.8, 102.5)
- moved J6 6.29 mm to (158.0, 109.6)
- moved D8 6.17 mm to (149.9, 109.0)
- moved R21 6.17 mm to (149.9, 105.0), turned to -90 degrees
- moved J3 3.56 mm to (139.5, 82.9)
- moved D7 3.43 mm to (150.2, 96.2)
- moved J5 3.43 mm to (158.1, 96.9)
- moved R20 3.43 mm to (150.3, 92.3)
- moved D4 2.67 mm to (150.2, 84.1)
- moved J4 2.67 mm to (158.2, 84.7)
- moved R19 2.67 mm to (150.2, 80.2), turned to -90 degrees
- moved R14 0.18 mm to (136.2, 106.0)
- moved R9 0.10 mm to (130.6, 87.7)
- moved R13 0.08 mm to (134.6, 86.6)
- moved R10 0.06 mm to (132.7, 88.4)
Connections:
- J6 pad 4: INT3 -> INT5
- J6 pad 6: RST3 -> RST5
- J6 pad 8: CS4 -> CS1
- J9 pad 4: INT5 -> INT3
- J9 pad 6: RST5 -> RST3
- R15 pad 1: CS1 -> unconnected-(R15-Pad1)
- U4 pad 12: RST5 -> INT5
- U4 pad 13: INT5 -> RST5
- U4 pad 23: CS2 -> RST1
- U4 pad 24: RST1 -> CS2
Routing:
- net SCK: track 0.00 -> 164.6 mm
- net MOSI: track 0.00 -> 139.9 mm
- net MISO: track 0.00 -> 132.7 mm, vias 0 -> 1
- net USBVCC: track 0.00 -> 58.7 mm
- net CS2: track 0.00 -> 52.7 mm, vias 0 -> 1
- net CS3: track 0.00 -> 43.1 mm, vias 0 -> 2
- net +3V3: track 0.00 -> 42.9 mm
- net RESET: track 0.00 -> 40.5 mm
- net CS1: track 0.00 -> 33.5 mm, vias 0 -> 1
- net RST5: track 0.00 -> 30.3 mm, vias 0 -> 1
- net RST1: track 0.00 -> 30.1 mm, vias 0 -> 1
- net INT1: track 0.00 -> 29.6 mm, vias 0 -> 1
- net RST2: track 0.00 -> 29.3 mm, vias 0 -> 1
- net RESET2: track 0.00 -> 28.2 mm
- net MISO_1: track 0.00 -> 27.0 mm, vias 0 -> 2
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
Commit message: routage bien avancé, derniers changement d'E/S sur le 328 pour faciliter le routage
Connections:
- J6 pad 4: INT5 -> INT3
- J6 pad 6: RST5 -> RST3
- J6 pad 8: CS1 -> CS4
- J9 pad 4: INT3 -> INT5
- J9 pad 6: RST3 -> RST5
- R15 pad 1: unconnected-(R15-Pad1) -> CS1
- R2 pad 1: CS4 -> CS1
- U4 pad 1: INT3 -> RST5
- U4 pad 10: INT4 -> RST4
- U4 pad 11: CS6 -> CS5
- U4 pad 12: INT5 -> INT3
- U4 pad 13: RST5 -> RST3
- U4 pad 14: CS1 -> CS4
- U4 pad 2: CS5 -> CS6
- U4 pad 30: CS4 -> CS1
- U4 pad 32: RST3 -> INT5
- U4 pad 9: RST4 -> INT4
Routing:
- net CS6: track 0.00 -> 34.6 mm, vias 0 -> 1
- net RST3: track 0.00 -> 30.3 mm, vias 0 -> 1
- net CS5: track 0.00 -> 29.4 mm, vias 0 -> 1
- net RST4: track 0.00 -> 28.6 mm, vias 0 -> 1
- net CS4: track 5.88 -> 33.5 mm, vias 0 -> 1
- net CS1: track 33.5 -> 5.88 mm, vias 1 -> 0
- net INT4: track 0.00 -> 27.5 mm, vias 0 -> 1
- net INT3: track 0.00 -> 26.5 mm
- net INT5: track 26.5 -> 39.3 mm, vias 0 -> 1
- net RST5: track 30.3 -> 36.1 mm

Commit message: routage presque terminé
Routing:
- net USBVCC: track 58.7 -> 239.7 mm, vias 0 -> 1
- net CS6: track 34.6 -> 66.6 mm, vias 1 -> 3
- net CS1: track 5.88 -> 31.2 mm, vias 0 -> 2
- net SCK_1: track 0.00 -> 19.2 mm, vias 0 -> 2
- net RESET: track 40.5 -> 58.3 mm, vias 0 -> 2
- net CS5: track 29.4 -> 36.6 mm
- net CS4: track 33.5 -> 37.6 mm, vias 1 -> 3
- net Net-(U4-XTAL1/PB6): track 15.1 -> 14.3 mm
- net MISO_1: track 27.0 -> 27.6 mm

Commit message: routage terminé, 24 erreur de DRC
Connections:
- U4 pad 21: Net-(U4-GND-Pad21) -> GND
- U4 pad 3: Net-(U4-GND-Pad21) -> GND
- U4 pad 5: Net-(U4-GND-Pad21) -> GND
Routing:
- net USBVCC: track 239.7 -> 283.9 mm, vias 1 -> 3
- net GND: track 2.71 -> 14.3 mm, vias 0 -> 52
- net +3V3: track 42.9 -> 51.3 mm, vias 0 -> 2
- added copper zone on B.Cu, net GND
- added copper zone on F.Cu, net GND
Other:
- board outline added: 73.6 x 51.9 mm

Commit message: modif schema et routage
Parts:
- moved C9 17.2 mm to (108.8, 85.2), turned to 0 degrees
- moved C13 7.99 mm to (116.8, 101.9), turned to 90 degrees
- moved C11 7.94 mm to (124.5, 101.7), turned to -90 degrees
- moved C2 4.58 mm to (132.2, 105.8)
- moved R4 4.12 mm to (110.0, 95.5)
- moved R3 3.92 mm to (110.0, 90.2)
- moved U2 3.56 mm to (133.1, 108.6)
- moved R14 2.85 mm to (139.0, 106.4), turned to 0 degrees
- moved R8 2.76 mm to (123.2, 81.4)
- moved SW1 2.53 mm to (142.0, 112.0)
- moved C3 2.53 mm to (133.0, 111.5)
- moved C6 2.14 mm to (138.0, 100.3)
- moved J9 1.97 mm to (104.1, 92.6)
- moved R12 1.86 mm to (112.8, 93.8)
- moved R13 1.65 mm to (135.0, 85.0), turned to 0 degrees
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- renumbered J4 to J1, J5 to J2, J6 to J3, J7 to J4, J9 to J5, J2 to J6, J3 to J7, J1 to J8, J8 to J9
Connections:
- net CS1_1 renamed CS_SD_3v3
- J1 pad 8: CS2 -> CS1
- J2 pad 8: CS3 -> CS2
- J3 pad 8: CS4 -> CS3
- J4 pad 8: CS5 -> CS4
- J5 pad 8: CS6 -> CS5
- R15 pad 1: CS1 -> CS_SD
- R19 pad 1: CS2 -> CS1
- R2 pad 1: CS1 -> CS_SD
- R20 pad 1: CS3 -> CS2
- R21 pad 1: CS4 -> CS3
- R22 pad 1: CS5 -> CS4
- R23 pad 1: CS6 -> CS5
- U4 pad 11: CS5 -> CS4
- U4 pad 14: CS4 -> CS3
- U4 pad 2: CS6 -> CS5
- U4 pad 24: CS2 -> CS1
- U4 pad 26: CS3 -> CS2
- U4 pad 30: CS1 -> CS_SD
Routing:
- net GND: track 14.3 -> 89.9 mm, vias 52 -> 78
- net CS6: track 66.6 -> 0.00 mm, vias 3 -> 0
- net CS_SD: track 0.00 -> 29.8 mm, vias 0 -> 2
- net CS5: track 36.6 -> 60.3 mm, vias 1 -> 3
- net SCK: track 164.6 -> 149.4 mm
- net USBVCC: track 283.9 -> 298.3 mm, vias 3 -> 6
- net RESET: track 58.3 -> 46.3 mm
- net CS2: track 52.7 -> 42.4 mm, vias 1 -> 2
- net CS1: track 31.2 -> 40.3 mm
- net RESET2: track 28.2 -> 19.5 mm
- net +3V3: track 51.3 -> 44.9 mm, vias 2 -> 4
- net CS3: track 43.1 -> 36.9 mm, vias 2 -> 3
- net Net-(U5-PC0/XTAL2): track 12.3 -> 6.97 mm
- net Net-(J9-D--PadA7): track 2.45 -> 5.99 mm
- net Net-(U4-XTAL1/PB6): track 14.3 -> 10.7 mm
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Other:
- board size 73.6 x 51.9 mm -> 73.5 x 52 mm
- board text added: "2024"
- board text added: "22R"
- board text added: "328p"
- board text added: "5k1"
- board text added: "8u2"
- board text added: "CS1"
- board text added: "CS2"
- board text added: "CS3"
- board text added: "CS4"
- board text added: "CS5"
- board text added: "GND"
- board text added: "INT1"
- board text added: "INT2"
- board text added: "INT3"
- board text added: "INT4"
- board text added: "INT5"
- board text added: "J1"
- board text added: "J2"
- board text added: "J3"
- board text added: "J4"
- board text added: "J5"
- board text added: "Louis Antoine"
- board text added: "MISO"
- board text added: "MOSI"
- board text added: "ON"
- board text added: "PicoMother"
- board text added: "RST"
- board text added: "RST 328p"
- board text added: "RST1"
- board text added: "RST2"
- board text added: "RST3"
- board text added: "RST4"
- board text added: "RST5"
- board text added: "RX"
- board text added: "SCK"
- board text added: "TX"
- board text added: "VCC"

Commit message: correction DRC
Parts:
- moved R5 0.24 mm to (132.0, 97.8)
Other:
- board text added: "16MHz"
Changed lines of the file:
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@@
 	(footprint "Resistor_SMD:R_0603_1608Metric_Pad0.98x0.95mm_HandSolder"
 		(layer "F.Cu")
-		(at 132.0311 98.044)
+		(at 132.0311 97.8)
 		(descr "Resistor SMD 0603 (1608 Metric), square (rectangular) end terminal, IPC_7351 nominal with elongated pad for handsoldering. (Body size source: IPC-SM-782 page 72, https://www.pcb-3d.com/wordpress/wp-content/uploads/ipc-sm-782a_amendment_1_and_2.pdf), generated with kicad-footprint-generator")
 		(tags "resistor handsolder")
@@
 		)
 	)
+	(gr_text "16MHz"
+		(at 118.4 105.2 0)
+		(layer "F.SilkS")
+		(effects
+			(font
+				(size 1 1)
+				(thickness 0.2)
+				(bold yes)
+			)
+			(justify left bottom)
+		)
+	)
 	(gr_text "22R"
 		(at 111.75 95.5 0)
@@
 		)
 	)
+	(gr_text "16MHz"
+		(at 141.2 105.6 0)
+		(layer "F.SilkS")
+		(effects
+			(font
+				(size 1 1)
+				(thickness 0.2)
+				(bold yes)
+			)
+			(justify left bottom)
+		)
+	)
 	(gr_text "22R"
 		(at 111.75 91.25 0)
@@
 	)
 	(segment
-		(start 132.9436 98.044)
-		(end 134.239 98.044)
+		(start 134 97.8)
+		(end 135.1788 96.6212)
 		(width 0.2)
 		(layer "F.Cu")
@@
 	)
 	(segment
-		(start 134.239 98.044)
-		(end 135.1788 97.1042)
+		(start 135.1788 96.6212)
+		(end 135.1788 94.6404)
 		(width 0.2)
 		(layer "F.Cu")
@@
 	)
 	(segment
-		(start 135.1788 97.1042)
-		(end 135.1788 94.6404)
+		(start 135.1788 94.6404)
+		(end 135.6874 94.1318)
 		(width 0.2)
 		(layer "F.Cu")
@@
 	)
 	(segment
-		(start 135.1788 94.6404)
-		(end 135.6874 94.1318)
+		(start 132.9436 97.8)
+		(end 134 97.8)
 		(width 0.2)
 		(layer "F.Cu")
@@
 	)
 	(segment
-		(start 131.1186 98.044)
-		(end 130.2512 98.044)
+		(start 128.5912 96.384)
+		(end 130.0072 97.8)
 		(width 0.2)
 		(layer "F.Cu")
@@
 	)
 	(segment
-		(start 130.2512 98.044)
-		(end 128.5912 96.384)
+		(start 130.0072 97.8)
+		(end 131.1186 97.8)
 		(width 0.2)
 		(layer "F.Cu")

Commit message: PCB terminé
Parts:
- moved D8 0.40 mm to (151.2, 109.9)
- moved R7 0.35 mm to (143.5, 98.4)
- moved Y1 0.34 mm to (143.6, 101.7)
- moved C11 0.25 mm to (124.5, 101.9)
- moved D7 0.20 mm to (151.2, 97.2)
- moved C5 0.15 mm to (147.4, 101.9)
- moved C4 0.09 mm to (139.8, 101.9)
Connections:
- net MISO_1 renamed MISO_3v3
- net MOSI_1 renamed MOSI_3v3
- net SCK_1 renamed SCK_3v3
Routing:
- net GND: track 89.9 -> 116.3 mm, vias 78 -> 94
- net CS2: track 42.4 -> 35.2 mm
- net MOSI: track 138.0 -> 132.4 mm
- net MISO: track 130.6 -> 126.4 mm, vias 1 -> 2
- net USBVCC: track 298.3 -> 300.6 mm
- net SCK: track 149.4 -> 147.9 mm
- net CS1: track 40.3 -> 39.6 mm
- net CS3: track 36.9 -> 36.3 mm
- net Net-(U4-XTAL1/PB6): track 10.7 -> 10.1 mm
- net CS5: track 60.3 -> 59.8 mm
Other:
- board text added: "CS_SD -> PD0"
- board text added: "Louis & Antoine"
- board text added: "RST1-> PC0 CS1 -> PC1 INT1-> PC2"
- board text added: "RST2-> PC4 CS2 -> PC3 INT2-> PC5"
- board text added: "RST3-> PB1 CS3 -> PB2 INT3-> PB0"
- board text added: "RST4-> PD6 CS4 -> PD7 INT4-> PD5"
- board text added: "RST5-> PD3 CS5 -> PD4 INT5-> PD2"
- board text removed: "Louis Antoine"
