File: PicoMother/PicoMother.kicad_pcb (KiCad board)
At the start: 2 copper layers, 73.5 x 52 mm, 57 parts, among them J1 Conn_02x04_Counter_Clockwise, J2 Conn_02x04_Counter_Clockwise, J3 Conn_02x04_Counter_Clockwise, J4 Conn_02x04_Counter_Clockwise, J5 Conn_02x04_Counter_Clockwise, J6 Micro_SD, J7 M20-9980345, J8 M20-9980345, J9 USB_C, SW1 SW_Push, U1 74LVC125, U2 LM1117-3.3, U4 ATmega328P-A, U5 ATmega8U2-A, Y1 Crystal_GND24, Y4 Crystal_GND24

Commit message: Generation fichiers gerber
Parts:
- moved R12 0.25 mm to (112.8, 93.5)
Routing:
- net INT4: track 27.6 -> 29.5 mm
- net RST4: track 28.6 -> 30.2 mm
- net CS4: track 37.0 -> 38.2 mm
- net RESET: track 46.3 -> 47.2 mm
- net MOSI: track 132.4 -> 133.1 mm
- net SCK: track 147.9 -> 148.4 mm
- net GND: vias 94 -> 96

Commit message: Correction inversion D+ D-
Parts:
- moved R11 1.82 mm to (114.2, 93.1), turned to 45 degrees
- moved C7 1.03 mm to (116.8, 89.8), turned to -90 degrees
- moved R12 0.97 mm to (112.2, 92.7), turned to 45 degrees
Connections:
- U5 pad 29: D- -> D+
- U5 pad 30: D+ -> D-
Routing:
- net GND: track 116.3 -> 131.0 mm
- net Net-(J9-D--PadA7): track 5.99 -> 7.93 mm
- net D+: track 5.40 -> 6.75 mm
- net D-: track 5.56 -> 4.75 mm
