File: PicoMother/ATMEGA328P-MU.kicad_sch (KiCad schematic)
At the start: 15 parts, among them J3 M20-9980345, SW1 SW_Push, U4 ATMEGA328P-MU, Y1 CSTNE16M0V530000R0

Commit message: avancement schema
Connections:
- net A0 renamed CS2
- net A1 renamed RST1
- net A2 renamed INT1
- net A3 renamed CS3
- net A4/SDA renamed RST2
- net A5/SCL renamed INT2
- net IO0: no longer names the net of R5.1, U4.30 (PD0)
- net IO1 renamed CS4
- net IO2 renamed RST3
- net IO3 renamed INT3
- net IO4 renamed CS5
- net IO5 renamed RST4
- net IO6 renamed INT4
- net IO7 renamed CS6
- net IO8 renamed RST5
- net IO9 renamed INT5
- net SS renamed CS1

Commit message: Schema PicoMother
Parts:
- removed D2: CD1206-S01575, Diode_SMD:D_1206_3216Metric, symbol Device:D
- removed FB2: 10uH, Inductor_SMD:L_0805_2012Metric, symbol Device:FerriteBead
- C1, C12, C7, C8: footprint Capacitor_SMD:C_0603_1608Metric -> Capacitor_SMD:C_0603_1608Metric_Pad1.08x0.95mm_HandSolder
- R2: footprint Resistor_SMD:R_0603_1608Metric -> Resistor_SMD:R_0603_1608Metric_Pad0.98x0.95mm_HandSolder; now fitted
- Y1: value CSTNE16M0V530000R0 -> 16Mhz; footprint Crystal:Resonator_SMD_Murata_CSTxExxV-3Pin_3.0x1.1mm -> Crystal:Crystal_SMD_SeikoEpson_FA238-4Pin_3.2x2.5mm_HandSoldering
Other:
- note added: "Empreinte ?"
- moved on the sheet: C1, C12, C7, C8, J3, R13, R14, SW1

Commit message: Premier Schema
Connections:
- net AREF: no longer names the net of C1.1, U4.20 (AREF)
- net AVCC: no longer names the net of C12.1, U4.18 (AVCC)
Other:
- note added: "AtMega 328p"
- note added: "ISP 328p"
- moved on the sheet: C1, C12, C7, C8, J3, R13, R14, R2, R5, R7, SW1, U4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

Commit message: correction schematique quartz
Parts:
- removed Y1: 16Mhz, Crystal:Crystal_SMD_SeikoEpson_FA238-4Pin_3.2x2.5mm_HandSoldering, symbol Device:Crystal_GND2
- added C4, C5: 22p, Capacitor_SMD:C_0603_1608Metric_Pad1.08x0.95mm_HandSolder, symbol Device:C
- added Y3: Crystal_GND24, Crystal:Crystal_SMD_SeikoEpson_FA238-4Pin_3.2x2.5mm_HandSoldering, symbol Device:Crystal_GND24
Connections:
- net GND: now also C4.2, C5.2, Y3.2, Y3.4
- net at R2.1, U4.8 (PB7): now also C4.1, Y3.3
- net at R2.2, U4.7 (PB6): now also C5.1, Y3.1
Other:
- moved on the sheet: C1, C12

Commit message: correction schematique empreintes MCU
Parts:
- removed C12, C7, C8: 100n, Capacitor_SMD:C_0603_1608Metric_Pad1.08x0.95mm_HandSolder, symbol Device:C
- removed U4: ATMEGA328P-MU, Package_QFP:TQFP-32_7x7mm_P0.8mm, symbol Arduino Uno SMD:ATMEGA328P-MU
- removed Y3: Crystal_GND24, Crystal:Crystal_SMD_SeikoEpson_FA238-4Pin_3.2x2.5mm_HandSoldering, symbol Device:Crystal_GND24
- added C6: 100n, Capacitor_SMD:C_0603_1608Metric_Pad1.08x0.95mm_HandSolder, symbol Device:C
- added U4: ATmega328P-A, Package_QFP:TQFP-32_7x7mm_P0.8mm, symbol MCU_Microchip_ATmega:ATmega328P-A
- added Y1: Crystal_GND24, Crystal:Crystal_SMD_SeikoEpson_FA238-4Pin_3.2x2.5mm_HandSoldering, symbol Device:Crystal_GND24
- R2: value 1M -> 1k
- R7: value 1k -> 1M
- SW1: footprint Button_Switch_THT:SW_DIP_SPSTx01_Piano_10.8x4.1mm_W7.62mm_P2.54mm -> Button_Switch_SMD:SW_Push_1P1T_NO_CK_KSC7xxJ
Connections:
- net +5V: now also C6.2, U4.18 (AVCC), U4.4 (VCC), U4.6 (VCC)
- net CS1: now also U4.14 (PB2)
- net CS2: now also U4.23 (PC0)
- net CS3: now also U4.26 (PC3)
- net CS4: now also R2.1, U4.30 (PD0); no longer R7.2
- net CS5: now also U4.2 (PD4)
- net CS6: now also U4.11 (PD7)
- net DTR: now also C1.1
- net GND: now also C6.1, Y1.2, Y1.4; no longer C1.2
- net INT1: now also U4.25 (PC2)
- net INT2: now also U4.28 (PC5)
- net INT3: now also U4.1 (PD3)
- net INT4: now also U4.10 (PD6)
- net INT5: now also U4.13 (PB1)
- net M8RXD: now also R2.2; no longer R5.2
- net M8TXD: now also R5.1; no longer R7.1
- net MISO: now also U4.16 (PB4)
- net MOSI: now also U4.15 (PB3)
- net RESET: now also C1.2, U4.29 (~{RESET}/PC6)
- net RST1: now also U4.24 (PC1)
- net RST2: now also U4.27 (PC4)
- net RST3: now also U4.32 (PD2)
- net RST4: now also U4.9 (PD5)
- net RST5: now also U4.12 (PB0)
- net SCK: now also U4.17 (PB5)
- net at C4.1: now also R7.1, U4.7 (XTAL1/PB6), Y1.3; no longer R2.1
- net at C5.1: now also R7.2, U4.8 (XTAL2/PB7), Y1.1; no longer R2.2
- new net: U4.21 (GND), U4.3 (GND), U4.5 (GND)
- new net: R5.2, U4.31 (PD1)
Other:
- note removed: "Empreinte ?"

Commit message: début de routage, premiers changement d'E/S sur le 328 pour faciliter le routage
Connections:
- net CS2: now also U4.24 (PC1); no longer U4.23 (PC0)
- net INT5: now also U4.12 (PB0); no longer U4.13 (PB1)
- net RST1: now also U4.23 (PC0); no longer U4.24 (PC1)
- net RST5: now also U4.13 (PB1); no longer U4.12 (PB0)

Commit message: routage bien avancé, derniers changement d'E/S sur le 328 pour faciliter le routage
Connections:
- net CS1: now also R2.1, U4.30 (PD0); no longer U4.14 (PB2)
- net CS4: now also U4.14 (PB2); no longer R2.1, U4.30 (PD0)
- net CS5: now also U4.11 (PD7); no longer U4.2 (PD4)
- net CS6: now also U4.2 (PD4); no longer U4.11 (PD7)
- net INT3: now also U4.12 (PB0); no longer U4.1 (PD3)
- net INT4: now also U4.9 (PD5); no longer U4.10 (PD6)
- net INT5: now also U4.32 (PD2); no longer U4.12 (PB0)
- net RST3: now also U4.13 (PB1); no longer U4.32 (PD2)
- net RST4: now also U4.10 (PD6); no longer U4.9 (PD5)
- net RST5: now also U4.1 (PD3); no longer U4.13 (PB1)

Commit message: routage terminé, 24 erreur de DRC
Connections:
- net GND: now also U4.21 (GND), U4.3 (GND), U4.5 (GND)
Changed lines of the file:
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@@
+	(symbol
+		(lib_id "power:GND")
+		(at 104.14 127 0)
+		(unit 1)
+		(exclude_from_sim no)
+		(in_bom yes)
+		(on_board yes)
+		(dnp no)
+		(fields_autoplaced yes)
+		(property "Reference" "#PWR044"
+			(at 104.14 133.35 0)
+			(effects
+				(font
+					(size 1.27 1.27)
+				)
+				(hide yes)
+			)
+		)
+		(property "Value" "GND"
+			(at 104.14 132.08 0)
+			(effects
+				(font
+					(size 1.27 1.27)
+				)
+			)
+		)
+		(property "Footprint" ""
+			(at 104.14 127 0)
+			(effects
+				(font
+					(size 1.27 1.27)
+				)
+				(hide yes)
+			)
+		)
+		(property "Datasheet" ""
+			(at 104.14 127 0)
+			(effects
+				(font
+					(size 1.27 1.27)
+				)
+				(hide yes)
+			)
+		)
+		(property "Description" "Power symbol creates a global label with name \"GND\" , ground"
+			(at 104.14 127 0)
+			(effects
+				(font
+					(size 1.27 1.27)
+				)
+				(hide yes)
+			)
+		)
+		(pin "1"
+		)
+		(instances
+			(project ""
+				(path "/a569fb01-6252-4b3a-9dcb-3675b5ce6f3f/2d22e81c-5a17-48ca-8b8a-97f7d3a7b1e3"
+					(reference "#PWR044")
+					(unit 1)
+				)
+			)
+		)
+	)
 	(symbol
 		(lib_id "power:GND")
