File: PicoMother/ATMEGA328P-MU.kicad_sch (KiCad schematic)
At the start: 13 parts, among them J3 M20-9980345, SW1 SW_Push, U4 ATmega328P-A, Y1 Crystal_GND24

Commit message: modif schema et routage
Parts:
- renumbered J3 to J7
Connections:
- net CS6 is gone; now on net CS5: U4.2 (PD4)
- net CS1: now also U4.24 (PC1); no longer R2.1, U4.30 (PD0)
- net CS2: now also U4.26 (PC3); no longer U4.24 (PC1)
- net CS3: now also U4.14 (PB2); no longer U4.26 (PC3)
- net CS4: now also U4.11 (PD7); no longer U4.14 (PB2)
- net CS5: no longer U4.11 (PD7)
- new net CS_SD: R2.1, U4.30 (PD0)
- no-connect marks 2 -> 3

Commit message: PCB terminé
Other:
- moved on the sheet: C6
Changed lines of the file:
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@@
 	(symbol
 		(lib_id "power:+5V")
-		(at 158.75 50.8 0)
+		(at 185.42 62.23 0)
 		(unit 1)
 		(exclude_from_sim no)
@@
 		(dnp no)
 		(property "Reference" "#PWR041"
-			(at 158.75 54.61 0)
+			(at 185.42 66.04 0)
 			(effects
 				(font
@@
 		)
 		(property "Value" "+5V"
-			(at 161.798 48.768 0)
+			(at 188.468 60.198 0)
 			(effects
 				(font
@@
 		)
 		(property "Footprint" ""
-			(at 158.75 50.8 0)
+			(at 185.42 62.23 0)
 			(effects
 				(font
@@
 		)
 		(property "Datasheet" ""
-			(at 158.75 50.8 0)
+			(at 185.42 62.23 0)
 			(effects
 				(font
@@
 		)
 		(property "Description" "Power symbol creates a global label with name \"+5V\""
-			(at 158.75 50.8 0)
+			(at 185.42 62.23 0)
 			(effects
 				(font
@@
 	(symbol
 		(lib_id "Device:C")
-		(at 158.75 54.61 180)
+		(at 185.42 66.04 180)
 		(unit 1)
 		(exclude_from_sim no)
@@
 		(dnp no)
 		(property "Reference" "C6"
-			(at 152.908 55.89 0)
+			(at 179.578 67.32 0)
 			(effects
 				(font
@@
 		)
 		(property "Value" "100n"
-			(at 152.908 53.34 0)
+			(at 179.578 64.77 0)
 			(effects
 				(font
@@
 		)
 		(property "Footprint" "Capacitor_SMD:C_0603_1608Metric_Pad1.08x0.95mm_HandSolder"
-			(at 157.7848 50.8 0)
+			(at 184.4548 62.23 0)
 			(effects
 				(font
@@
 		)
 		(property "Datasheet" "~"
-			(at 158.75 54.61 0)
+			(at 185.42 66.04 0)
 			(effects
 				(font
@@
 		)
 		(property "Description" "Unpolarized capacitor"
-			(at 158.75 54.61 0)
+			(at 185.42 66.04 0)
 			(effects
 				(font
@@
 	(symbol
 		(lib_id "power:GND")
-		(at 158.75 58.42 0)
+		(at 185.42 69.85 0)
 		(unit 1)
 		(exclude_from_sim no)
@@
 		(fields_autoplaced yes)
 		(property "Reference" "#PWR042"
-			(at 158.75 64.77 0)
+			(at 185.42 76.2 0)
 			(effects
 				(font
@@
 		)
 		(property "Value" "GND"
-			(at 158.75 63.5 0)
+			(at 185.42 74.93 0)
 			(effects
 				(font
@@
 		)
 		(property "Footprint" ""
-			(at 158.75 58.42 0)
+			(at 185.42 69.85 0)
 			(effects
 				(font
@@
 		)
 		(property "Datasheet" ""
-			(at 158.75 58.42 0)
+			(at 185.42 69.85 0)
 			(effects
 				(font
@@
 		)
 		(property "Description" "Power symbol creates a global label with name \"GND\" , ground"
-			(at 158.75 58.42 0)
-			(effects
-				(font
+			(at 185.42 69.85 0)
+			(effects
+				(font
