File: PicoMother/ATMEGA328P-MU.kicad_sch (KiCad schematic)
At the start: 13 parts, among them J7 M20-9980345, SW1 SW_Push, U4 ATmega328P-A, Y1 Crystal_GND24

Commit message: correction CS SD
Connections:
- net CS3: now also R2.1, U4.30 (PD0); no longer U4.14 (PB2)
- net CS_SD: now also U4.14 (PB2); no longer R2.1, U4.30 (PD0)
