File: PicoMother/PicoMother.kicad_sch (KiCad schematic)
At the start: 24 parts, among them J1 M20-9980345, J8 USB_C_Receptacle_USB2.0_16P, U3 ATMEGA16U2-MU, Y2 LFXTAL003240BULK

Commit message: avancement schema
Other:
- moved on the sheet: D1, R6
Changed lines of the file:
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@@
 	(wire
 		(pts
-			(xy 229.87 83.82) (xy 229.87 78.74)
+			(xy 204.47 93.98) (xy 204.47 88.9)
 		)
 		(stroke
@@
 	(wire
 		(pts
-			(xy 261.62 83.82) (xy 256.54 83.82)
+			(xy 236.22 93.98) (xy 231.14 93.98)
 		)
 		(stroke
@@
 	(wire
 		(pts
-			(xy 229.87 83.82) (xy 234.95 83.82)
+			(xy 204.47 93.98) (xy 209.55 93.98)
 		)
 		(stroke
@@
 	(wire
 		(pts
-			(xy 242.57 83.82) (xy 248.92 83.82)
+			(xy 217.17 93.98) (xy 223.52 93.98)
 		)
 		(stroke
@@
 	(symbol
 		(lib_id "Device:R")
-		(at 238.76 83.82 90)
+		(at 213.36 93.98 90)
 		(unit 1)
 		(exclude_from_sim no)
@@
 		(fields_autoplaced yes)
 		(property "Reference" "R6"
-			(at 238.76 77.47 90)
+			(at 213.36 87.63 90)
 			(effects
 				(font
@@
 		)
 		(property "Value" "2k"
-			(at 238.76 80.01 90)
+			(at 213.36 90.17 90)
 			(effects
 				(font
@@
 		)
 		(property "Footprint" "Resistor_SMD:R_0603_1608Metric_Pad0.98x0.95mm_HandSolder"
-			(at 238.76 85.598 90)
+			(at 213.36 95.758 90)
 			(effects
 				(font
@@
 		)
 		(property "Datasheet" "~"
-			(at 238.76 83.82 0)
+			(at 213.36 93.98 0)
 			(effects
 				(font
@@
 		)
 		(property "Description" "Resistor"
-			(at 238.76 83.82 0)
+			(at 213.36 93.98 0)
 			(effects
 				(font
@@
 	(symbol
 		(lib_id "power:+5V")
-		(at 229.87 78.74 0)
+		(at 204.47 88.9 0)
 		(unit 1)
 		(exclude_from_sim no)
@@
 		(fields_autoplaced yes)
 		(property "Reference" "#PWR01"
-			(at 229.87 82.55 0)
+			(at 204.47 92.71 0)
 			(effects
 				(font
@@
 		)
 		(property "Value" "+5V"
-			(at 229.87 73.66 0)
+			(at 204.47 83.82 0)
 			(effects
 				(font
@@
 		)
 		(property "Footprint" ""
-			(at 229.87 78.74 0)
+			(at 204.47 88.9 0)
 			(effects
 				(font
@@
 		)
 		(property "Datasheet" ""
-			(at 229.87 78.74 0)
+			(at 204.47 88.9 0)
 			(effects
 				(font
@@
 		)
 		(property "Description" "Power symbol creates a global label with name \"+5V\""
-			(at 229.87 78.74 0)
+			(at 204.47 88.9 0)
 			(effects
 				(font
@@
 	(symbol
 		(lib_id "Device:LED")
-		(at 252.73 83.82 180)
+		(at 227.33 93.98 180)
 		(unit 1)
 		(exclude_from_sim no)
@@
 		(fields_autoplaced yes)
 		(property "Reference" "D1"
-			(at 254.3175 76.2 0)
+			(at 228.9175 86.36 0)
 			(effects
 				(font
@@
 		)
 		(property "Value" "GREEN"
-			(at 254.3175 78.74 0)
+			(at 228.9175 88.9 0)
 			(effects
 				(font
@@
 		)
 		(property "Footprint" "LED_SMD:LED_0805_2012Metric"
-			(at 252.73 83.82 0)
+			(at 227.33 93.98 0)
 			(effects
 				(font
@@
 		)
 		(property "Datasheet" "~"
-			(at 252.73 83.82 0)
+			(at 227.33 93.98 0)
 			(effects
 				(font
@@
 		)
 		(property "Description" "Light emitting diode"
-			(at 252.73 83.82 0)
+			(at 227.33 93.98 0)
 			(effects
 				(font
@@
 	(symbol
 		(lib_id "power:GND")
-		(at 261.62 83.82 90)
+		(at 236.22 93.98 90)
 		(unit 1)
 		(exclude_from_sim no)
@@
 		(fields_autoplaced yes)
 		(property "Reference" "#PWR02"
-			(at 267.97 83.82 0)
+			(at 242.57 93.98 0)
 			(effects
 				(font
@@
 		)
 		(property "Value" "GND"
-			(at 265.43 83.8199 90)
+			(at 240.03 93.9799 90)
 			(effects
 				(font
@@
 		)
 		(property "Footprint" ""
-			(at 261.62 83.82 0)
+			(at 236.22 93.98 0)
 			(effects
 				(font
@@
 		)
 		(property "Datasheet" ""
-			(at 261.62 83.82 0)
+			(at 236.22 93.98 0)
 			(effects
 				(font
@@
 		)
 		(property "Description" "Power symbol creates a global label with name \"GND\" , ground"
-			(at 261.62 83.82 0)
+			(at 236.22 93.98 0)
 			(effects
 				(font

Commit message: Schema PicoMother
Parts:
- removed D3: CD1206-S01575, Diode_SMD:D_1206_3216Metric, symbol Device:D
- removed FB1: 1kΩ@100MHz, Inductor_SMD:L_0805_2012Metric, symbol Device:FerriteBead
- removed Z1, Z2: 5pF@1MHz, Resistor_SMD:R_0603_1608Metric, symbol Device:Varistor
- C10, C11, C13, C9: footprint Capacitor_SMD:C_0603_1608Metric -> Capacitor_SMD:C_0603_1608Metric_Pad1.08x0.95mm_HandSolder
- D1, D5, D6: footprint LED_SMD:LED_0805_2012Metric -> LED_SMD:LED_0603_1608Metric_Pad1.05x0.95mm_HandSolder
- J8: value USB_C_Receptacle_USB2.0_16P -> USB_C
- R1: footprint Resistor_SMD:R_0603_1608Metric -> Resistor_SMD:R_0603_1608Metric_Pad0.98x0.95mm_HandSolder; now fitted
- R3, R4: footprint Resistor_SMD:R_0603_1608Metric -> Resistor_SMD:R_0603_1608Metric_Pad0.98x0.95mm_HandSolder
- U3: value ATMEGA16U2-MU -> ATMEGA8U2-MU
- Y2: value LFXTAL003240BULK -> 16Mhz; footprint Crystal:Crystal_HC49-4H_Vertical -> Crystal:Crystal_SMD_SeikoEpson_FA238-4Pin_3.2x2.5mm_HandSoldering
Connections:
- net USHIELD is gone; now on net GND: J8.S1 (SHIELD)
Other:
- note added: "ISP 8u2"
- note added: "LEDS"
- note added: "USB C"
- moved on the sheet: C10, C11, C13, C9, D1, D5, D6, J1, J8, R10, R11, R12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

Commit message: Premier Schema
Parts:
- D1: value GREEN -> LED
- D5, D6: value YELLOW -> LED
Connections:
- net RD+ is gone; now on net D+: R12.2, U3.29 (D+)
- net RD- is gone; now on net D-: R11.2, U3.30 (D-)
- net +5V: now also J8.A4 (VBUS), J8.A9 (VBUS), J8.B4 (VBUS), J8.B9 (VBUS); no longer J1.2 (Pin_2)
- net D+: no longer J8.A6 (D+), J8.B6 (D+), R12.1
- net D-: no longer J8.A7 (D-), J8.B7 (D-), R11.1
- net GND: now also D1.2 (A); no longer D1.1 (K)
- net RESET2: now also J1.2 (Pin_2)
- net USBVCC: no longer J8.A4 (VBUS), J8.A9 (VBUS), J8.B4 (VBUS), J8.B9 (VBUS)
- net at R6.2: now also D1.1 (K); no longer D1.2 (A)
- new net: J8.A7 (D-), J8.B7 (D-), R11.1
- new net: J8.A6 (D+), J8.B6 (D+), R12.1
- no-connect marks 11 -> 15
Other:
- note added: "AtMega8u2"
- moved on the sheet: C9, D1, J8, R11, R12, R3, R4, R8

Commit message: correction schematique quartz
Parts:
- removed Y2: 16Mhz, Crystal:Crystal_SMD_SeikoEpson_FA238-4Pin_3.2x2.5mm_HandSoldering, symbol Device:Crystal
- added Y4: Crystal_GND24, Crystal:Crystal_SMD_SeikoEpson_FA238-4Pin_3.2x2.5mm_HandSoldering, symbol Device:Crystal_GND24
Connections:
- net GND: now also Y4.2, Y4.4
- net at C13.1, R1.1, U3.2 (PC0): now also Y4.3
- net at C11.1, R1.2, U3.1 (XTAL1): now also Y4.1
Other:
- moved on the sheet: C13
Changed lines of the file:
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@@
 	)
 	(junction
+		(at 138.43 114.3)
+		(diameter 0)
+		(color 0 0 0 0)
+	)
+	(junction
 		(at 153.67 125.73)
 		(diameter 0)
@@
 	)
 	(junction
-		(at 138.43 106.68)
+		(at 152.4 151.13)
 		(diameter 0)
 		(color 0 0 0 0)
 	)
 	(junction
-		(at 152.4 151.13)
+		(at 123.19 116.84)
 		(diameter 0)
 		(color 0 0 0 0)
 	)
 	(junction
-		(at 123.19 116.84)
+		(at 59.69 115.57)
 		(diameter 0)
 		(color 0 0 0 0)
 	)
 	(junction
-		(at 138.43 114.3)
+		(at 123.19 110.49)
 		(diameter 0)
 		(color 0 0 0 0)
 	)
 	(junction
-		(at 59.69 115.57)
+		(at 123.19 104.14)
 		(diameter 0)
 		(color 0 0 0 0)
@@
 		(color 0 0 0 0)
 	)
+	(junction
+		(at 138.43 106.68)
+		(diameter 0)
+		(color 0 0 0 0)
+	)
 	(no_connect
 		(at 186.69 95.25)
@@
 	(wire
 		(pts
+			(xy 123.19 104.14) (xy 123.19 110.49)
+		)
+		(stroke
+			(width 0)
+			(type default)
+		)
+	)
+	(wire
+		(pts
 			(xy 147.32 143.51) (xy 156.21 143.51)
 		)
@@
 	(wire
 		(pts
-			(xy 123.19 102.87) (xy 124.46 102.87)
+			(xy 123.19 100.33) (xy 124.46 100.33)
 		)
 		(stroke
@@
 		)
 	)
+	(wire
+		(pts
+			(xy 123.19 110.49) (xy 123.19 116.84)
+		)
+		(stroke
+			(width 0)
+			(type default)
+		)
+	)
 	(polyline
 		(pts
@@
 	(wire
 		(pts
+			(xy 123.19 110.49) (xy 133.35 110.49)
+		)
+		(stroke
+			(width 0)
+			(type default)
+		)
+	)
+	(wire
+		(pts
 			(xy 147.32 140.97) (xy 156.21 140.97)
 		)
@@
 	(wire
 		(pts
-			(xy 138.43 106.68) (xy 138.43 102.87)
+			(xy 138.43 106.68) (xy 138.43 100.33)
 		)
 		(stroke
@@
 		)
 	)
+	(wire
+		(pts
+			(xy 143.51 110.49) (xy 143.51 104.14)
+		)
+		(stroke
+			(width 0)
+			(type default)
+		)
+	)
 	(polyline
 		(pts
@@
 	(wire
 		(pts
-			(xy 123.19 102.87) (xy 123.19 116.84)
+			(xy 123.19 100.33) (xy 123.19 104.14)
 		)
 		(stroke
@@
 	(wire
 		(pts
-			(xy 138.43 102.87) (xy 132.08 102.87)
+			(xy 138.43 100.33) (xy 132.08 100.33)
 		)
 		(stroke
@@
 	(wire
 		(pts
+			(xy 123.19 104.14) (xy 143.51 104.14)
+		)
+		(stroke
+			(width 0)
+			(type default)
+		)
+	)
+	(wire
+		(pts
 			(xy 138.43 116.84) (xy 138.43 114.3)
 		)
@@
 	(symbol
 		(lib_id "Device:C")
-		(at 128.27 102.87 270)
+		(at 128.27 100.33 270)
 		(unit 1)
 		(exclude_from_sim no)
@@
 		(dnp no)
 		(property "Reference" "C13"
-			(at 127 97.028 0)
+			(at 128.524 97.028 90)
 			(effects
 				(font
@@
 		)
 		(property "Value" "22p"
-			(at 129.54 97.028 0)
+			(at 128.524 94.488 90)
 			(effects
 				(font
@@
 		)
 		(property "Footprint" "Capacitor_SMD:C_0603_1608Metric_Pad1.08x0.95mm_HandSolder"
-			(at 124.46 103.8352 0)
+			(at 124.46 101.2952 0)
 			(effects
 				(font
@@
 		)
 		(property "Datasheet" "~"
-			(at 128.27 102.87 0)
+			(at 128.27 100.33 0)
 			(effects
 				(font
@@
 		)
 		(property "Description" "Unpolarized capacitor"
-			(at 128.27 102.87 0)
+			(at 128.27 100.33 0)
 			(effects
 				(font
@@
 	)
 	(symbol
-		(lib_id "Device:Crystal")
-		(at 138.43 110.49 270)
-		(unit 1)
-		(exclude_from_sim no)
-		(in_bom yes)
-		(on_board yes)
-		(dnp no)
-		(fields_autoplaced yes)
-		(property "Reference" "Y2"
-			(at 142.24 109.2199 90)
-			(effects
-				(font
-					(size 1.27 1.27)
-				)
-				(justify left)
-			)
-		)
-		(property "Value" "16Mhz"
-			(at 142.24 111.7599 90)
-			(effects
-				(font
-					(size 1.27 1.27)
-				)
-				(justify left)
-				(hide yes)
-			)
-		)
-		(property "Footprint" "Crystal:Crystal_SMD_SeikoEpson_FA238-4Pin_3.2x2.5mm_HandSoldering"
-			(at 138.43 110.49 0)
-			(effects
-				(font
-					(size 1.27 1.27)
-				)
-				(hide yes)
-			)
-		)
-		(property "Datasheet" "~"
-			(at 138.43 110.49 0)
-			(effects
-				(font
-					(size 1.27 1.27)
-				)
-				(hide yes)
-			)
-		)
-		(property "Description" "Two pin crystal"
-			(at 138.43 110.49 0)
-			(effects
-				(font
-					(size 1.27 1.27)
-				)
-				(hide yes)
-			)
-		)
-		(pin "1"
-		)
-		(pin "2"
-		)
-		(instances
-			(project "Arduino Uno SMD"
-				(path "/a569fb01-6252-4b3a-9dcb-3675b5ce6f3f"
-					(reference "Y2")
-					(unit 1)
-				)
-			)
-		)
-	)
-	(symbol
 		(lib_id "power:GND")
 		(at 152.4 153.67 0)
@@
 	)
 	(symbol
+		(lib_id "Device:Crystal_GND24")
+		(at 138.43 110.49 90)
+		(unit 1)
+		(exclude_from_sim no)
+		(in_bom yes)
+		(on_board yes)
+		(dnp no)
+		(fields_autoplaced yes)
+		(property "Reference" "Y4"
+			(at 144.78 108.0768 90)
+			(effects
+				(font
+					(size 1.27 1.27)
+				)
+			)
+		)
+		(property "Value" "Crystal_GND24"
+			(at 151.13 108.0768 90)
+			(effects
+				(font
+					(size 1.27 1.27)
+				)
+				(hide yes)
+			)
+		)
+		(property "Footprint" "Crystal:Crystal_SMD_SeikoEpson_FA238-4Pin_3.2x2.5mm_HandSoldering"
+			(at 138.43 110.49 0)
+			(effects
+				(font
+					(size 1.27 1.27)
+				)
+				(hide yes)
+			)
+		)
+		(property "Datasheet" "~"
+			(at 138.43 110.49 0)
+			(effects
+				(font
+					(size 1.27 1.27)
+				)
+				(hide yes)
+			)
+		)
+		(property "Description" "Four pin crystal, GND on pins 2 and 4"
+			(at 138.43 110.49 0)
+			(effects
+				(font
+					(size 1.27 1.27)
+				)
+				(hide yes)
+			)
+		)
+		(pin "3"
+		)
+		(pin "2"
+		)
+		(pin "1"
+		)
+		(pin "4"
+		)
+		(instances
+			(project ""
+				(path "/a569fb01-6252-4b3a-9dcb-3675b5ce6f3f"
+					(reference "Y4")
+					(unit 1)
+				)
+			)
+		)
+	)
+	(symbol
 		(lib_id "Device:LED")
 		(at 219.71 55.88 0)
@@
 		(dnp no)
 		(property "Reference" "C11"
-			(at 127 110.998 0)
+			(at 128.524 122.682 90)
 			(effects
 				(font
@@
 		)
 		(property "Value" "22p"
-			(at 129.54 110.998 0)
+			(at 128.524 120.142 90)
 			(effects
 				(font

Commit message: correction schematique reset
Connections:
- net +5V: now also J1.2 (Pin_2)
- net RESET2: no longer J1.2 (Pin_2)
Changed lines of the file:
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@@
 	)
 	(junction
-		(at 160.02 50.8)
-		(diameter 0)
-		(color 0 0 0 0)
-	)
-	(junction
 		(at 152.4 151.13)
 		(diameter 0)
@@
 	(wire
 		(pts
-			(xy 160.02 50.8) (xy 167.64 50.8)
+			(xy 157.48 50.8) (xy 157.48 48.26)
 		)
 		(stroke
@@
 	(wire
 		(pts
-			(xy 149.86 50.8) (xy 160.02 50.8)
-		)
-		(stroke
-			(width 0)
-			(type default)
-		)
-	)
-	(wire
-		(pts
 			(xy 156.21 128.27) (xy 152.4 128.27)
 		)
@@
 	(wire
 		(pts
-			(xy 153.67 125.73) (xy 156.21 125.73)
+			(xy 149.86 50.8) (xy 157.48 50.8)
 		)
 		(stroke
@@
 	(wire
 		(pts
-			(xy 160.02 49.53) (xy 160.02 50.8)
+			(xy 153.67 125.73) (xy 156.21 125.73)
 		)
 		(stroke
@@
 		)
 	)
-	(global_label "RESET2"
-		(shape input)
-		(at 167.64 50.8 0)
-		(fields_autoplaced yes)
-		(effects
-			(font
-				(size 1.27 1.27)
-			)
-			(justify left)
-		)
-		(property "Intersheetrefs" "${INTERSHEET_REFS}"
-			(at 177.5798 50.8 0)
-			(effects
-				(font
-					(size 1.27 1.27)
-				)
-				(justify left)
-				(hide yes)
-			)
-		)
-	)
 	(global_label "RXLED"
 		(shape input)
@@
 	(symbol
 		(lib_id "power:+5V")
-		(at 160.02 41.91 0)
-		(unit 1)
-		(exclude_from_sim no)
-		(in_bom yes)
-		(on_board yes)
-		(dnp no)
-		(fields_autoplaced yes)
-		(property "Reference" "#PWR025"
-			(at 160.02 45.72 0)
-			(effects
-				(font
-					(size 1.27 1.27)
-				)
-				(hide yes)
-			)
-		)
-		(property "Value" "+5V"
-			(at 160.02 36.83 0)
-			(effects
-				(font
-					(size 1.27 1.27)
-				)
-			)
-		)
-		(property "Footprint" ""
-			(at 160.02 41.91 0)
-			(effects
-				(font
-					(size 1.27 1.27)
-				)
-				(hide yes)
-			)
-		)
-		(property "Datasheet" ""
-			(at 160.02 41.91 0)
-			(effects
-				(font
-					(size 1.27 1.27)
-				)
-				(hide yes)
-			)
-		)
-		(property "Description" "Power symbol creates a global label with name \"+5V\""
-			(at 160.02 41.91 0)
-			(effects
-				(font
-					(size 1.27 1.27)
-				)
-				(hide yes)
-			)
-		)
-		(pin "1"
-		)
-		(instances
-			(project "Arduino Uno SMD"
-				(path "/a569fb01-6252-4b3a-9dcb-3675b5ce6f3f"
-					(reference "#PWR025")
-					(unit 1)
-				)
-			)
-		)
-	)
-	(symbol
-		(lib_id "power:+5V")
 		(at 72.39 102.87 0)
 		(unit 1)
@@
 	)
 	(symbol
+		(lib_id "power:+5V")
+		(at 157.48 48.26 0)
+		(unit 1)
+		(exclude_from_sim no)
+		(in_bom yes)
+		(on_board yes)
+		(dnp no)
+		(fields_autoplaced yes)
+		(property "Reference" "#PWR043"
+			(at 157.48 52.07 0)
+			(effects
+				(font
+					(size 1.27 1.27)
+				)
+				(hide yes)
+			)
+		)
+		(property "Value" "+5V"
+			(at 157.48 43.18 0)
+			(effects
+				(font
+					(size 1.27 1.27)
+				)
+			)
+		)
+		(property "Footprint" ""
+			(at 157.48 48.26 0)
+			(effects
+				(font
+					(size 1.27 1.27)
+				)
+				(hide yes)
+			)
+		)
+		(property "Datasheet" ""
+			(at 157.48 48.26 0)
+			(effects
+				(font
+					(size 1.27 1.27)
+				)
+				(hide yes)
+			)
+		)
+		(property "Description" "Power symbol creates a global label with name \"+5V\""
+			(at 157.48 48.26 0)
+			(effects
+				(font
+					(size 1.27 1.27)
+				)
+				(hide yes)
+			)
+		)
+		(pin "1"
+		)
+		(instances
+			(project "PicoMother"
+				(path "/a569fb01-6252-4b3a-9dcb-3675b5ce6f3f"
+					(reference "#PWR043")
+					(unit 1)
+				)
+			)
+		)
+	)
+	(symbol
 		(lib_id "Device:R")
 		(at 73.66 146.05 0)
@@
 	)
 	(symbol
-		(lib_id "Device:R")
-		(at 160.02 45.72 0)
-		(unit 1)
-		(exclude_from_sim no)
-		(in_bom yes)
-		(on_board yes)
-		(dnp no)
-		(fields_autoplaced yes)
-		(property "Reference" "R8"
-			(at 162.56 44.4499 0)
-			(effects
-				(font
-					(size 1.27 1.27)
-				)
-				(justify left)
-			)
-		)
-		(property "Value" "10k"
-			(at 162.56 46.9899 0)
-			(effects
-				(font
-					(size 1.27 1.27)
-				)
-				(justify left)
-			)
-		)
-		(property "Footprint" "Resistor_SMD:R_0603_1608Metric_Pad0.98x0.95mm_HandSolder"
-			(at 158.242 45.72 90)
-			(effects
-				(font
-					(size 1.27 1.27)
-				)
-				(hide yes)
-			)
-		)
-		(property "Datasheet" "~"
-			(at 160.02 45.72 0)
-			(effects
-				(font
-					(size 1.27 1.27)
-				)
-				(hide yes)
-			)
-		)
-		(property "Description" "Resistor"
-			(at 160.02 45.72 0)
-			(effects
-				(font
-					(size 1.27 1.27)
-				)
-				(hide yes)
-			)
-		)
-		(pin "2"
-		)
-		(pin "1"
-		)
-		(instances
-			(project ""
-				(path "/a569fb01-6252-4b3a-9dcb-3675b5ce6f3f"
-					(reference "R8")
-					(unit 1)
-				)
-			)
-		)
-	)
-	(symbol
 		(lib_id "power:GND")
 		(at 152.4 153.67 0)
@@
 	)
 	(symbol
+		(lib_id "Device:R")
+		(at 156.21 96.52 0)
+		(unit 1)
+		(exclude_from_sim no)
+		(in_bom yes)
+		(on_board yes)
+		(dnp no)
+		(fields_autoplaced yes)
+		(property "Reference" "R8"
+			(at 158.75 95.2499 0)
+			(effects
+				(font
+					(size 1.27 1.27)
+				)
+				(justify left)
+			)
+		)
+		(property "Value" "10k"
+			(at 158.75 97.7899 0)
+			(effects
+				(font
+					(size 1.27 1.27)
+				)
+				(justify left)
+			)
+		)
+		(property "Footprint" "Resistor_SMD:R_0603_1608Metric_Pad0.98x0.95mm_HandSolder"
+			(at 154.432 96.52 90)
+			(effects
+				(font
+					(size 1.27 1.27)
+				)
+				(hide yes)
+			)
+		)
+		(property "Datasheet" "~"
+			(at 156.21 96.52 0)
+			(effects
+				(font
+					(size 1.27 1.27)
+				)
+				(hide yes)
+			)
+		)
+		(property "Description" "Resistor"
+			(at 156.21 96.52 0)
+			(effects
+				(font
+					(size 1.27 1.27)
+				)
+				(hide yes)
+			)
+		)
+		(pin "2"
+		)
+		(pin "1"
+		)
+		(instances
+			(project "PicoMother"
+				(path "/a569fb01-6252-4b3a-9dcb-3675b5ce6f3f"
+					(reference "R8")
+					(unit 1)
+				)
+			)
+		)
+	)
+	(symbol
 		(lib_id "power:GND")
 		(at 240.03 36.83 0)
@@
 					(unit 1)
 				)
+			)
+		)
+	)
+	(symbol
+		(lib_id "power:+5V")
+		(at 156.21 92.71 0)
+		(unit 1)
+		(exclude_from_sim no)
+		(in_bom yes)
+		(on_board yes)
+		(dnp no)
+		(fields_autoplaced yes)
+		(property "Reference" "#PWR025"
+			(at 156.21 96.52 0)
+			(effects
+				(font
+					(size 1.27 1.27)
+				)
+				(hide yes)
+			)
+		)
+		(property "Value" "+5V"
+			(at 156.21 87.63 0)
+			(effects
+				(font
+					(size 1.27 1.27)
+				)
+			)
+		)
+		(property "Footprint" ""
+			(at 156.21 92.71 0)
+			(effects
+				(font
+					(size 1.27 1.27)
+				)
+				(hide yes)
+			)
+		)
+		(property "Datasheet" ""
+			(at 156.21 92.71 0)
+			(effects
+				(font
+					(size 1.27 1.27)
+				)
+				(hide yes)
+			)
+		)
+		(property "Description" "Power symbol creates a global label with name \"+5V\""
+			(at 156.21 92.71 0)
+			(effects
+				(font
+					(size 1.27 1.27)
+				)
+				(hide yes)
+			)
+		)
+		(pin "1"
+		)
+		(instances
+			(project "PicoMother"
+				(path "/a569fb01-6252-4b3a-9dcb-3675b5ce6f3f"
+					(reference "#PWR025")
+					(unit 1)
+				)

Commit message: correction schematique empreintes MCU
Parts:
- removed C10: 1u, Capacitor_SMD:C_0603_1608Metric_Pad1.08x0.95mm_HandSolder, symbol Device:C
- removed U3: ATMEGA8U2-MU, Package_QFP:TQFP-32_7x7mm_P0.8mm, symbol Arduino Uno SMD:ATMEGA16U2-MU
- added C7: 1u, Capacitor_SMD:C_0603_1608Metric_Pad1.08x0.95mm_HandSolder, symbol Device:C
- added U5: ATmega8U2-A, Package_QFP:TQFP-32_7x7mm_P0.8mm, symbol MCU_Microchip_ATmega:ATmega8U2-A
Connections:
- net +5V: now also U5.31 (UVCC), U5.32 (AVCC), U5.4 (VCC)
- net D+: now also U5.30 (D-)
- net D-: now also U5.29 (D+)
- net DTR: now also U5.13 (~{HWB}/PD7)
- net GND: now also C7.1, U5.28 (UGND), U5.3 (GND)
- net M8RXD: now also U5.9 (PD3)
- net M8TXD: now also U5.8 (PD2)
- net MISO2: now also U5.17 (PB3)
- net MOSI2: now also U5.16 (PB2)
- net RESET2: now also U5.24 (PC1/~{RESET})
- net RXLED: now also U5.10 (PD4)
- net SCK2: now also U5.15 (PB1)
- net TXLED: now also U5.11 (PD5)
- net at C13.1, R1.1, Y4.3: now also U5.1 (XTAL1)
- net at C11.1, R1.2, Y4.1: now also U5.2 (PC0/XTAL2)
- new net: C7.2, U5.27 (UCAP)
Other:
- moved on the sheet: C11, C13, D1, D5, D6, J1, R1, R10, R6, R9, Y4

Commit message: modif schema et routage
Parts:
- renumbered J1 to J8, J8 to J9
Changed lines of the file:
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@@
+	)
+	(junction
+		(at 121.92 93.98)
+		(diameter 0)
+		(color 0 0 0 0)
 	)
 	(junction
@@
 	)
 	(junction
-		(at 121.92 92.71)
-		(diameter 0)
-		(color 0 0 0 0)
-	)
-	(junction
 		(at 39.37 140.97)
 		(diameter 0)
@@
 	(wire
 		(pts
-			(xy 121.92 92.71) (xy 121.92 99.06)
-		)
-		(stroke
-			(width 0)
-			(type default)
-		)
-	)
-	(wire
-		(pts
 			(xy 137.16 95.25) (xy 146.05 95.25)
 		)
@@
 	(wire
 		(pts
+			(xy 121.92 93.98) (xy 121.92 99.06)
+		)
+		(stroke
+			(width 0)
+			(type default)
+		)
+	)
+	(wire
+		(pts
 			(xy 242.57 39.37) (xy 242.57 45.72)
 		)
@@
 	(wire
 		(pts
-			(xy 142.24 99.06) (xy 142.24 92.71)
+			(xy 142.24 99.06) (xy 142.24 93.98)
 		)
 		(stroke
@@
 	(wire
 		(pts
-			(xy 121.92 88.9) (xy 121.92 92.71)
+			(xy 121.92 88.9) (xy 121.92 93.98)
 		)
 		(stroke
@@
 	(wire
 		(pts
-			(xy 121.92 92.71) (xy 142.24 92.71)
+			(xy 121.92 93.98) (xy 142.24 93.98)
 		)
 		(stroke
@@
 		(dnp no)
 		(fields_autoplaced yes)
-		(property "Reference" "J8"
+		(property "Reference" "J9"
 			(at 43.18 95.25 0)
 			(effects
@@
 			(project "Arduino Uno SMD"
 				(path "/a569fb01-6252-4b3a-9dcb-3675b5ce6f3f"
-					(reference "J8")
+					(reference "J9")
 					(unit 1)
 				)
@@
 		(dnp no)
 		(fields_autoplaced yes)
-		(property "Reference" "J1"
+		(property "Reference" "J8"
 			(at 143.51 34.29 0)
 			(effects
@@
 			(project "Arduino Uno SMD"
 				(path "/a569fb01-6252-4b3a-9dcb-3675b5ce6f3f"
-					(reference "J1")
+					(reference "J8")
 					(unit 1)
 				)
