File: PicoMother/Connectors.kicad_sch (KiCad schematic)
At the start: 22 parts, among them J2 Micro_SD_Card_Det2, J4 Conn_02x04_Counter_Clockwise, J5 Conn_02x04_Counter_Clockwise, J6 Conn_02x04_Counter_Clockwise, J7 Conn_02x04_Counter_Clockwise, J9 Conn_02x04_Counter_Clockwise, U1 74LVC125

Commit message: avancement schema
Parts:
- removed C6: 100n, Capacitor_SMD:C_0603_1608Metric, symbol Device:C
Connections:
- no-connect marks 5 -> 4
Other:
- note added: "Ajouter regulateur 3V3"

Commit message: Schema PicoMother
Parts:
- added C2, C3: 100nF, Capacitor_SMD:C_0603_1608Metric_Pad1.08x0.95mm_HandSolder, symbol Device:C
- added U2: LM1117-3.3, Package_TO_SOT_SMD:SOT-23, symbol Regulator_Linear:LM1117-3.3
- J2: value Micro_SD_Card_Det2 -> Micro_SD
Connections:
- net +3V3: now also C3.1, U2.2 (VO)
- net +5V: now also C2.1, U2.3 (VI)
- net GND: now also C2.2, C3.2, U2.1 (GND)
Other:
- note added: "Connecteur SD"
- note added: "Régulateur 3v3"
- note removed: "Ajouter regulateur 3V3"
- note removed: "Lecteur SD"

Commit message: Premier Schema
Other:
- note added: "Conversion niveaux logiques SD"
- note removed: "Conversion niveaux logiques"
- moved on the sheet: C2, C3, J2, R15, R16, R17, R18, U1A, U1B, U1C, U1D, U1E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

Commit message: début de routage, premiers changement d'E/S sur le 328 pour faciliter le routage
Connections:
- net CS1: now also J6.8 (Pin_8); no longer R15.1
- net CS4: no longer J6.8 (Pin_8)
- net INT3: now also J9.4 (Pin_4); no longer J6.4 (Pin_4)
- net INT5: now also J6.4 (Pin_4); no longer J9.4 (Pin_4)
- net RST3: now also J9.6 (Pin_6); no longer J6.6 (Pin_6)
- net RST5: now also J6.6 (Pin_6); no longer J9.6 (Pin_6)

Commit message: routage bien avancé, derniers changement d'E/S sur le 328 pour faciliter le routage
Connections:
- net CS1: now also R15.1; no longer J6.8 (Pin_8)
- net CS4: now also J6.8 (Pin_8)
- net INT3: now also J6.4 (Pin_4); no longer J9.4 (Pin_4)
- net INT5: now also J9.4 (Pin_4); no longer J6.4 (Pin_4)
- net RST3: now also J6.6 (Pin_6); no longer J9.6 (Pin_6)
- net RST5: now also J9.6 (Pin_6); no longer J6.6 (Pin_6)

Commit message: modif schema et routage
Parts:
- renumbered J4 to J1, J5 to J2, J6 to J3, J7 to J4, J9 to J5, J2 to J6
Connections:
- net CS6 is gone; now on net CS5: J5.8 (Pin_8), R23.1
- net CS1: now also J1.8 (Pin_8), R19.1; no longer R15.1
- net CS2: now also J2.8 (Pin_8), R20.1; no longer J1.8 (Pin_8), R19.1
- net CS3: now also J3.8 (Pin_8), R21.1; no longer J2.8 (Pin_8), R20.1
- net CS4: now also J4.8 (Pin_8), R22.1; no longer J3.8 (Pin_8), R21.1
- net CS5: no longer J4.8 (Pin_8), R22.1
- net CS1_1 renamed CS_SD_3v3
- new net CS_SD: R15.1
Changed lines of the file:
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@@
 		)
 	)
-	(global_label "CS4"
+	(global_label "CS3"
 		(shape input)
 		(at 171.45 123.19 0)
@@
 		)
 		(property "Intersheetrefs" "${INTERSHEET_REFS}"
-			(at 178.0448 123.19 0)
+			(at 178.1242 123.19 0)
 			(effects
 				(font
@@
 		)
 	)
-	(global_label "CS3"
+	(global_label "CS2"
 		(shape input)
 		(at 130.81 123.19 0)
@@
 		)
 		(property "Intersheetrefs" "${INTERSHEET_REFS}"
-			(at 137.4048 123.19 0)
+			(at 137.4842 123.19 0)
 			(effects
 				(font
@@
 		)
 	)
-	(global_label "CS6"
+	(global_label "CS5"
 		(shape input)
 		(at 251.46 123.19 0)
@@
 		)
 		(property "Intersheetrefs" "${INTERSHEET_REFS}"
-			(at 258.0548 123.19 0)
+			(at 258.1342 123.19 0)
 			(effects
 				(font
@@
 		)
 	)
-	(global_label "CS5"
+	(global_label "CS4"
 		(shape input)
 		(at 210.82 123.19 0)
@@
 		)
 		(property "Intersheetrefs" "${INTERSHEET_REFS}"
-			(at 217.4148 123.19 0)
+			(at 217.4942 123.19 0)
 			(effects
 				(font
@@
 		)
 	)
-	(global_label "CS3"
+	(global_label "CS2"
 		(shape input)
 		(at 118.11 144.78 180)
@@
 		)
 		(property "Intersheetrefs" "${INTERSHEET_REFS}"
-			(at 111.5152 144.78 0)
+			(at 111.4358 144.78 0)
 			(effects
 				(font
@@
 		)
 	)
-	(global_label "CS2"
+	(global_label "CS1"
 		(shape input)
 		(at 90.17 123.19 0)
@@
 		)
 		(property "Intersheetrefs" "${INTERSHEET_REFS}"
-			(at 96.7648 123.19 0)
+			(at 96.8442 123.19 0)
 			(effects
 				(font
@@
 		)
 	)
-	(global_label "CS2"
+	(global_label "CS1"
 		(shape input)
 		(at 77.47 144.78 180)
@@
 		)
 		(property "Intersheetrefs" "${INTERSHEET_REFS}"
-			(at 70.8752 144.78 0)
+			(at 70.7958 144.78 0)
 			(effects
 				(font
@@
 		)
 	)
-	(global_label "CS1"
+	(global_label "CS_SD"
 		(shape input)
 		(at 132.08 54.61 90)
@@
 		)
 		(property "Intersheetrefs" "${INTERSHEET_REFS}"
-			(at 132.08 47.9358 90)
+			(at 132.08 45.6982 90)
 			(effects
 				(font
@@
 		)
 	)
-	(global_label "CS1_1"
+	(global_label "CS_SD_3v3"
 		(shape input)
 		(at 218.44 48.26 180)
@@
 		)
 		(property "Intersheetrefs" "${INTERSHEET_REFS}"
-			(at 209.6681 48.26 0)
+			(at 205.174 48.26 0)
 			(effects
 				(font
@@
 		)
 	)
-	(global_label "CS5"
+	(global_label "CS4"
 		(shape input)
 		(at 198.12 144.78 180)
@@
 		)
 		(property "Intersheetrefs" "${INTERSHEET_REFS}"
-			(at 191.5252 144.78 0)
+			(at 191.4458 144.78 0)
 			(effects
 				(font
@@
 		)
 	)
-	(global_label "CS6"
+	(global_label "CS5"
 		(shape input)
 		(at 238.76 144.78 180)
@@
 		)
 		(property "Intersheetrefs" "${INTERSHEET_REFS}"
-			(at 232.1652 144.78 0)
+			(at 232.0858 144.78 0)
 			(effects
 				(font
@@
 		)
 	)
-	(global_label "CS4"
+	(global_label "CS3"
 		(shape input)
 		(at 158.75 144.78 180)
@@
 		)
 		(property "Intersheetrefs" "${INTERSHEET_REFS}"
-			(at 152.1552 144.78 0)
+			(at 152.0758 144.78 0)
 			(effects
 				(font
@@
 		)
 	)
-	(global_label "CS1_1"
+	(global_label "CS_SD_3v3"
 		(shape input)
 		(at 147.32 62.23 0)
@@
 		)
 		(property "Intersheetrefs" "${INTERSHEET_REFS}"
-			(at 156.0919 62.23 0)
+			(at 160.586 62.23 0)
 			(effects
 				(font
@@
 		(dnp no)
 		(fields_autoplaced yes)
-		(property "Reference" "J5"
-			(at 124.46 120.65 0)
+		(property "Reference" "J2"
+			(at 124.46 119.38 0)
 			(effects
 				(font
@@
 			(project "PicoMother"
 				(path "/a569fb01-6252-4b3a-9dcb-3675b5ce6f3f/6fd3874c-ab98-487b-bc14-add57500a864"
-					(reference "J5")
+					(reference "J2")
 					(unit 1)
 				)
@@
 		(dnp no)
 		(fields_autoplaced yes)
-		(property "Reference" "J2"
+		(property "Reference" "J6"
 			(at 241.935 34.29 0)
 			(effects
@@
 			(project "PicoMother"
 				(path "/a569fb01-6252-4b3a-9dcb-3675b5ce6f3f/6fd3874c-ab98-487b-bc14-add57500a864"
-					(reference "J2")
+					(reference "J6")
 					(unit 1)
 				)
@@
 		(dnp no)
 		(fields_autoplaced yes)
-		(property "Reference" "J9"
-			(at 245.11 120.65 0)
+		(property "Reference" "J5"
+			(at 245.11 119.38 0)
 			(effects
 				(font
@@
 			(project "PicoMother"
 				(path "/a569fb01-6252-4b3a-9dcb-3675b5ce6f3f/6fd3874c-ab98-487b-bc14-add57500a864"
-					(reference "J9")
+					(reference "J5")
 					(unit 1)
 				)
@@
 		(dnp no)
 		(fields_autoplaced yes)
-		(property "Reference" "J7"
-			(at 204.47 120.65 0)
+		(property "Reference" "J4"
+			(at 204.47 119.38 0)
 			(effects
 				(font
@@
 			(project "PicoMother"
 				(path "/a569fb01-6252-4b3a-9dcb-3675b5ce6f3f/6fd3874c-ab98-487b-bc14-add57500a864"
-					(reference "J7")
+					(reference "J4")
 					(unit 1)
 				)
@@
 		(dnp no)
 		(fields_autoplaced yes)
-		(property "Reference" "J4"
-			(at 83.82 120.65 0)
+		(property "Reference" "J1"
+			(at 83.82 119.38 0)
 			(effects
 				(font
@@
 			(project "PicoMother"
 				(path "/a569fb01-6252-4b3a-9dcb-3675b5ce6f3f/6fd3874c-ab98-487b-bc14-add57500a864"
-					(reference "J4")
+					(reference "J1")
 					(unit 1)
 				)
@@
 		(dnp no)
 		(fields_autoplaced yes)
-		(property "Reference" "J6"
-			(at 165.1 120.65 0)
+		(property "Reference" "J3"
+			(at 165.1 119.38 0)
 			(effects
 				(font
@@
 			(project "PicoMother"
 				(path "/a569fb01-6252-4b3a-9dcb-3675b5ce6f3f/6fd3874c-ab98-487b-bc14-add57500a864"
-					(reference "J6")
+					(reference "J3")
 					(unit 1)
 				)

Commit message: PCB terminé
Connections:
- net MISO_1 renamed MISO_3v3
- net MOSI_1 renamed MOSI_3v3
- net SCK_1 renamed SCK_3v3
Changed lines of the file:
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@@
 		)
 	)
-	(global_label "MOSI_1"
+	(global_label "MOSI_3v3"
 		(shape input)
 		(at 218.44 50.8 180)
@@
 		)
 		(property "Intersheetrefs" "${INTERSHEET_REFS}"
-			(at 208.7609 50.8 0)
-			(effects
-				(font
-					(size 1.27 1.27)
-				)
-				(justify right)
-				(hide yes)
-			)
-		)
-	)
-	(global_label "MISO_1"
+			(at 206.5044 50.8 0)
+			(effects
+				(font
+					(size 1.27 1.27)
+				)
+				(justify right)
+				(hide yes)
+			)
+		)
+	)
+	(global_label "MISO_3v3"
 		(shape input)
 		(at 163.83 55.88 90)
@@
 		)
 		(property "Intersheetrefs" "${INTERSHEET_REFS}"
-			(at 163.83 46.1215 90)
+			(at 163.83 43.9444 90)
 			(effects
 				(font
@@
 		)
 	)
-	(global_label "MOSI_1"
+	(global_label "MOSI_3v3"
 		(shape input)
 		(at 148.59 41.91 0)
@@
 		)
 		(property "Intersheetrefs" "${INTERSHEET_REFS}"
-			(at 158.2691 41.91 0)
+			(at 160.5256 41.91 0)
 			(effects
 				(font
@@
 		)
 	)
-	(global_label "MISO_1"
+	(global_label "MISO_3v3"
 		(shape input)
 		(at 218.44 60.96 180)
@@
 		)
 		(property "Intersheetrefs" "${INTERSHEET_REFS}"
-			(at 208.7609 60.96 0)
+			(at 206.5044 60.96 0)
 			(effects
 				(font
@@
 		)
 	)
-	(global_label "SCK_1"
+	(global_label "SCK_3v3"
 		(shape input)
 		(at 218.44 55.88 180)
@@
 		)
 		(property "Intersheetrefs" "${INTERSHEET_REFS}"
-			(at 209.6076 55.88 0)
+			(at 207.3511 55.88 0)
 			(effects
 				(font
@@
 		)
 	)
-	(global_label "SCK_1"
+	(global_label "SCK_3v3"
 		(shape input)
 		(at 179.07 41.91 0)
@@
 		)
 		(property "Intersheetrefs" "${INTERSHEET_REFS}"
-			(at 187.9024 41.91 0)
-			(effects
-				(font
+			(at 190.1589 41.91 0)
+			(effects
+				(font
